File: wearables/kicad/MTCH101_Disc.sch (KiCad schematic (older format))
At the start: 13 parts, among them U1 MTCH101

Commit message: more exploration
Parts:
- added P1: SNS, Pin_Headers:Pin_Header_Straight_2x02, symbol CONN_02X02
- added W2: TEST_GND, Measurement_Points:Measurement_Point_Round-TH_Big, symbol TEST_1P
- added W5: TEST_VDD, Measurement_Points:Measurement_Point_Round-TH_Big, symbol TEST_1P
- D1: footprint LEDs:LED_0603 -> LEDs:LED_1206
- W1: footprint Measurement_Points:Measurement_Point_Round-SMD-Pad_Small -> (none)
- W3, W4: footprint Measurement_Points:Measurement_Point_Round-SMD-Pad_Small -> Mounting_Holes:MountingHole_2.2mm_M2_Pad
Connections:
- wire segments 22 -> 30
Changed lines of the file:
@@
 F 0 "#vdd01" H 7000 2400 50  0001 C CNN
 F 1 "VDD" H 7000 2700 50  0000 C CNN
-F 2 "" H 7000 2550 50  0000 C CNN
+F 2 "" H 7000 2550 25  0000 C CNN
 F 3 "" H 7000 2550 50  0000 C CNN
 	1    7000 2550
@@
 L GND #gnd02
 U 1 1 58064CAC
-P 7000 3400
-F 0 "#gnd02" H 7000 3150 50  0001 C CNN
-F 1 "GND" H 7000 3250 50  0000 C CNN
-F 2 "" H 7000 3400 50  0000 C CNN
-F 3 "" H 7000 3400 50  0000 C CNN
-	1    7000 3400
+P 7000 3500
+F 0 "#gnd02" H 7000 3250 50  0001 C CNN
+F 1 "GND" H 7000 3350 50  0000 C CNN
+F 2 "" H 7000 3500 25  0000 C CNN
+F 3 "" H 7000 3500 50  0000 C CNN
+	1    7000 3500
 	1    0    0    -1
 $EndComp
@@
 	1    0    0    -1
 $EndComp
-Wire Wire Line
-	5300 3450 5300 3600
-Wire Wire Line
-	5300 4200 5300 4350
-Wire Wire Line
-	7000 3150 7000 3400
-Wire Wire Line
-	7000 2550 7000 2850
 $Comp
 L R R4
@@
 	-1   0    0    1
 $EndComp
-Wire Wire Line
-	5700 3800 6100 3800
 $Comp
 L R R1
@@
 	1    0    0    -1
 $EndComp
-Wire Wire Line
-	3500 2700 3500 2900
-Wire Wire Line
-	3500 2800 4500 2800
-Connection ~ 3500 2800
-Wire Wire Line
-	3500 2300 3500 2400
-Wire Wire Line
-	3500 3200 3500 3300
 $Comp
 L R R3
@@
 	0    1    1    0
 $EndComp
-Wire Wire Line
-	4800 2800 4800 3800
-Wire Wire Line
-	4800 3800 4900 3800
-Wire Wire Line
-	4900 4000 4600 4000
-Wire Wire Line
-	4300 4000 3700 4000
 $Comp
 L TEST_1P W1
@@
 F 0 "W1" H 3700 4270 50  0000 C CNN
 F 1 "TEST_MTI" H 3700 4200 50  0000 C CNN
-F 2 "Measurement_Points:Measurement_Point_Round-SMD-Pad_Small" H 3900 4000 50  0001 C CNN
+F 2 "" H 3900 4000 50  0001 C CNN
 F 3 "" H 3900 4000 50  0000 C CNN
 	1    3700 4000
@@
 F 0 "W3" H 4400 2970 50  0000 C CNN
 F 1 "TEST_MTSA" H 4400 2900 50  0000 C CNN
-F 2 "Measurement_Points:Measurement_Point_Round-SMD-Pad_Small" H 4600 2700 50  0001 C CNN
+F 2 "Mounting_Holes:MountingHole_2.2mm_M2_Pad" H 4600 2700 50  0001 C CNN
 F 3 "" H 4600 2700 50  0000 C CNN
 	1    4400 2700
@@
 F 0 "D1" H 6400 3400 50  0000 C CNN
 F 1 "LED" H 6400 3200 50  0000 C CNN
-F 2 "LEDs:LED_0603" H 6400 3300 50  0000 C TNN
+F 2 "LEDs:LED_1206" H 6400 3300 50  0000 C TNN
 F 3 "" H 6400 3300 50  0000 C CNN
 	1    6400 3300
 	0    -1   -1   0
 $EndComp
-Wire Wire Line
-	6400 4000 6400 3900
-Wire Wire Line
-	6400 3500 6400 3600
-Wire Wire Line
-	6400 2900 6400 3100
 $Comp
 L TEST_1P W4
@@
 F 0 "W4" H 6500 4270 50  0000 C CNN
 F 1 "TEST_MTO" H 6500 4200 50  0000 C CNN
-F 2 "Measurement_Points:Measurement_Point_Round-SMD-Pad_Small" H 6700 4000 50  0001 C CNN
+F 2 "Mounting_Holes:MountingHole_2.2mm_M2_Pad" H 6700 4000 50  0001 C CNN
 F 3 "" H 6700 4000 50  0000 C CNN
 	1    6500 4000
@@
 Text Label 4650 4000 0    60   ~ 0
 MTI
-Wire Wire Line
-	5700 4000 6500 4000
-Connection ~ 6400 4000
 Text Label 3900 4000 0    60   ~ 0
 sns
@@
 	0    1    1    0
 $EndComp
-Wire Wire Line
-	5900 3200 5900 3400
-Wire Wire Line
-	5900 3700 5900 3800
-Connection ~ 5900 3800
-Wire Wire Line
-	4400 2700 4400 2800
-Connection ~ 4400 2800
 $Comp
 L VDD #vdd03
@@
 	0    1    1    0
 $EndComp
+$Comp
+L CONN_02X02 P1
+U 1 1 580797CC
+P 3150 4050
+F 0 "P1" H 3150 4200 50  0000 C CNN
+F 1 "SNS" H 3150 3900 50  0000 C CNN
+F 2 "Pin_Headers:Pin_Header_Straight_2x02" H 3150 2850 50  0000 C CNN
+F 3 "" H 3150 2850 50  0000 C CNN
+	1    3150 4050
+	1    0    0    -1
+$EndComp
+Wire Wire Line
+	5300 3450 5300 3600
+Wire Wire Line
+	5300 4200 5300 4350
+Wire Wire Line
+	7000 3150 7000 3500
+Wire Wire Line
+	7000 2550 7000 2850
+Wire Wire Line
+	5700 3800 6100 3800
+Wire Wire Line
+	3500 2700 3500 2900
+Wire Wire Line
+	3500 2800 4500 2800
+Connection ~ 3500 2800
+Wire Wire Line
+	3500 2300 3500 2400
+Wire Wire Line
+	3500 3200 3500 3300
+Wire Wire Line
+	4800 2800 4800 3800
+Wire Wire Line
+	4800 3800 4900 3800
+Wire Wire Line
+	4900 4000 4600 4000
+Wire Wire Line
+	3400 4000 4300 4000
+Wire Wire Line
+	6400 4000 6400 3900
+Wire Wire Line
+	6400 3500 6400 3600
+Wire Wire Line
+	6400 2900 6400 3100
+Wire Wire Line
+	5700 4000 6500 4000
+Connection ~ 6400 4000
+Wire Wire Line
+	5900 3200 5900 3400
+Wire Wire Line
+	5900 3700 5900 3800
+Connection ~ 5900 3800
+Wire Wire Line
+	4400 2700 4400 2800
+Connection ~ 4400 2800
 Wire Wire Line
 	7150 2800 7000 2800
@@
 	7150 3300 7000 3300
 Connection ~ 7000 3300
+Connection ~ 3700 4000
+Wire Wire Line
+	3450 4000 3450 4250
+Wire Wire Line
+	3450 4100 3400 4100
+Connection ~ 3450 4000
+Wire Wire Line
+	3450 4250 2800 4250
+Wire Wire Line
+	2800 4250 2800 4000
+Wire Wire Line
+	2800 4000 2900 4000
+Connection ~ 3450 4100
+Wire Wire Line
+	2800 4100 2900 4100
+Connection ~ 2800 4100
+$Comp
+L TEST_1P W5
+U 1 1 5807E2FD
+P 6900 2600
+F 0 "W5" H 6900 2870 50  0000 C CNN
+F 1 "TEST_VDD" H 6900 2800 50  0000 C CNN
+F 2 "Measurement_Points:Measurement_Point_Round-TH_Big" H 7100 2600 50  0001 C CNN
+F 3 "" H 7100 2600 50  0000 C CNN
+	1    6900 2600
+	0    -1   -1   0
+$EndComp
+$Comp
+L TEST_1P W2
+U 1 1 5807E47E
+P 6900 3400
+F 0 "W2" H 6900 3670 50  0000 C CNN
+F 1 "TEST_GND" H 6900 3600 50  0000 C CNN
+F 2 "Measurement_Points:Measurement_Point_Round-TH_Big" H 7100 3400 50  0001 C CNN
+F 3 "" H 7100 3400 50  0000 C CNN
+	1    6900 3400
+	0    -1   -1   0
+$EndComp
+Wire Wire Line
+	6900 2600 7000 2600
+Connection ~ 7000 2600
+Wire Wire Line
+	6900 3400 7000 3400
+Connection ~ 7000 3400
 $EndSCHEMATC

Commit message: Creating button connector library
Parts:
- removed P1: SNS, Pin_Headers:Pin_Header_Straight_2x02, symbol CONN_02X02
- removed W1: TEST_MTI, symbol TEST_1P
- added W1: sns, buttons:sew_2x2, symbol SEW_2X2
- R2: value OPEN -> 100k
Connections:
- wire segments 30 -> 24
Changed lines of the file:
@@
 LIBS:valves
 LIBS:mtch101
+LIBS:buttons
 LIBS:MTCH101_Disc-cache
 EELAYER 25 0
@@
 P 3500 3050
 F 0 "R2" V 3580 3050 50  0000 C CNN
-F 1 "OPEN" V 3500 3050 50  0000 C CNN
+F 1 "100k" V 3500 3050 50  0000 C CNN
 F 2 "Resistors_SMD:R_0603_HandSoldering" H 3430 3050 50  0000 R CNN
 F 3 "" H 3500 3050 50  0000 C CNN
@@
 	1    4450 4000
 	0    1    1    0
-$EndComp
-$Comp
-L TEST_1P W1
-U 1 1 580654F7
-P 3700 4000
-F 0 "W1" H 3700 4270 50  0000 C CNN
-F 1 "TEST_MTI" H 3700 4200 50  0000 C CNN
-F 2 "" H 3900 4000 50  0001 C CNN
-F 3 "" H 3900 4000 50  0000 C CNN
-	1    3700 4000
-	1    0    0    -1
 $EndComp
 $Comp
@@
 	0    1    1    0
 $EndComp
-$Comp
-L CONN_02X02 P1
-U 1 1 580797CC
-P 3150 4050
-F 0 "P1" H 3150 4200 50  0000 C CNN
-F 1 "SNS" H 3150 3900 50  0000 C CNN
-F 2 "Pin_Headers:Pin_Header_Straight_2x02" H 3150 2850 50  0000 C CNN
-F 3 "" H 3150 2850 50  0000 C CNN
-	1    3150 4050
-	1    0    0    -1
-$EndComp
 Wire Wire Line
 	5300 3450 5300 3600
@@
 	4900 4000 4600 4000
 Wire Wire Line
-	3400 4000 4300 4000
-Wire Wire Line
 	6400 4000 6400 3900
 Wire Wire Line
@@
 	7150 3300 7000 3300
 Connection ~ 7000 3300
-Connection ~ 3700 4000
-Wire Wire Line
-	3450 4000 3450 4250
-Wire Wire Line
-	3450 4100 3400 4100
-Connection ~ 3450 4000
-Wire Wire Line
-	3450 4250 2800 4250
-Wire Wire Line
-	2800 4250 2800 4000
-Wire Wire Line
-	2800 4000 2900 4000
-Connection ~ 3450 4100
-Wire Wire Line
-	2800 4100 2900 4100
-Connection ~ 2800 4100
 $Comp
 L TEST_1P W5
@@
 	6900 3400 7000 3400
 Connection ~ 7000 3400
+$Comp
+L SEW_2X2 W1
+U 1 1 5808D751
+P 3700 4000
+F 0 "W1" H 3700 4270 50  0000 C CNN
+F 1 "sns" H 3700 4200 50  0000 C CNN
+F 2 "buttons:sew_2x2" H 3900 4000 50  0000 C CNN
+F 3 "" H 3900 4000 50  0000 C CNN
+	1    3700 4000
+	1    0    0    -1
+$EndComp
+Wire Wire Line
+	3700 4000 4300 4000
 $EndSCHEMATC

Commit message: reworking.
Parts:
- removed U1: MTCH101, TO_SOT_Packages_SMD:SOT-23-6, symbol MTCH101
- added U1: MTCH101_PKG, TO_SOT_Packages_SMD:SOT-23-6, symbol MTCH101_PKG
Connections:
- net GND: now also U1.2 (VSS)
- net MTI: now also U1.1 (MTI)
- net MTSA: now also U1.3 (MTSA)
- net VDD: now also U1.5 (VDD)
- net out: now also U1.4 (MTO)
- net pm: now also U1.6 (MTPM)
Other:
- moved on the sheet: D1, R1, R2, R3, R4, R5, R6, W1, W3, W4, W6

Commit message: more seweable terminal variants
Parts:
- removed W2: TEST_GND, Measurement_Points:Measurement_Point_Round-TH_Big, symbol TEST_1P
- removed W3: TEST_MTSA, Mounting_Holes:MountingHole_2.2mm_M2_Pad, symbol TEST_1P
- removed W4: TEST_MTO, Mounting_Holes:MountingHole_2.2mm_M2_Pad, symbol TEST_1P
- removed W5: TEST_VDD, Measurement_Points:Measurement_Point_Round-TH_Big, symbol TEST_1P
- added W2: gnd, buttons:sew_1x2, symbol SEW_1X2
- added W3: sa, buttons:sew_1x2, symbol SEW_1X2
- added W4: out, buttons:sew_1x2, symbol SEW_1X2
- added W5: vdd, buttons:sew_1x2, symbol SEW_1X2
Connections:
- net GND: now also W2.1
- net VDD: now also W5.1
- net out: now also W4.1
- net ref: now also W3.1
Changed lines of the file:
@@
-$EndComp
-$Comp
-L TEST_1P W3
-U 1 1 58065576
-P 2900 5400
-F 0 "W3" H 2900 5670 50  0000 C CNN
-F 1 "TEST_MTSA" H 2900 5600 50  0000 C CNN
-F 2 "Mounting_Holes:MountingHole_2.2mm_M2_Pad" H 3100 5400 50  0001 C CNN
-F 3 "" H 3100 5400 50  0000 C CNN
-	1    2900 5400
-	1    0    0    -1
 $EndComp
 $Comp
@@
 	1    5400 4900
 	0    -1   -1   0
-$EndComp
-$Comp
-L TEST_1P W4
-U 1 1 58065ACD
-P 5500 5600
-F 0 "W4" H 5500 5870 50  0000 C CNN
-F 1 "TEST_MTO" H 5500 5800 50  0000 C CNN
-F 2 "Mounting_Holes:MountingHole_2.2mm_M2_Pad" H 5700 5600 50  0001 C CNN
-F 3 "" H 5700 5600 50  0000 C CNN
-	1    5500 5600
-	0    1    1    0
 $EndComp
 Text Label 4950 5600 0    60   ~ 0
@@
 	7150 3300 7000 3300
 Connection ~ 7000 3300
-$Comp
-L TEST_1P W5
-U 1 1 5807E2FD
-P 6900 2600
-F 0 "W5" H 6900 2870 50  0000 C CNN
-F 1 "TEST_VDD" H 6900 2800 50  0000 C CNN
-F 2 "Measurement_Points:Measurement_Point_Round-TH_Big" H 7100 2600 50  0001 C CNN
-F 3 "" H 7100 2600 50  0000 C CNN
-	1    6900 2600
-	0    -1   -1   0
-$EndComp
-$Comp
-L TEST_1P W2
-U 1 1 5807E47E
-P 6900 3400
-F 0 "W2" H 6900 3670 50  0000 C CNN
-F 1 "TEST_GND" H 6900 3600 50  0000 C CNN
-F 2 "Measurement_Points:Measurement_Point_Round-TH_Big" H 7100 3400 50  0001 C CNN
-F 3 "" H 7100 3400 50  0000 C CNN
-	1    6900 3400
-	0    -1   -1   0
-$EndComp
 Wire Wire Line
 	6900 2600 7000 2600
@@
 Wire Wire Line
 	2900 5400 2900 5600
+$Comp
+L SEW_1X2 W3
+U 1 1 580A30E6
+P 2900 5400
+F 0 "W3" H 2900 5670 50  0000 C CNN
+F 1 "sa" H 2900 5600 50  0000 C CNN
+F 2 "buttons:sew_1x2" H 3100 5400 50  0000 C CNN
+F 3 "" H 3100 5400 50  0000 C CNN
+	1    2900 5400
+	1    0    0    -1
+$EndComp
+$Comp
+L SEW_1X2 W4
+U 1 1 580A3684
+P 5500 5600
+F 0 "W4" H 5500 5870 50  0000 C CNN
+F 1 "out" H 5500 5800 50  0000 C CNN
+F 2 "buttons:sew_1x2" H 5700 5600 50  0000 C CNN
+F 3 "" H 5700 5600 50  0000 C CNN
+	1    5500 5600
+	0    1    1    0
+$EndComp
+$Comp
+L SEW_1X2 W5
+U 1 1 580A4007
+P 6900 2600
+F 0 "W5" H 6900 2870 50  0000 C CNN
+F 1 "vdd" H 6900 2800 50  0000 C CNN
+F 2 "buttons:sew_1x2" H 7100 2600 50  0000 C CNN
+F 3 "" H 7100 2600 50  0000 C CNN
+	1    6900 2600
+	0    -1   -1   0
+$EndComp
+$Comp
+L SEW_1X2 W2
+U 1 1 580A4052
+P 6900 3400
+F 0 "W2" H 6900 3670 50  0000 C CNN
+F 1 "gnd" H 6900 3600 50  0000 C CNN
+F 2 "buttons:sew_1x2" H 7100 3400 50  0000 C CNN
+F 3 "" H 7100 3400 50  0000 C CNN
+	1    6900 3400
+	0    -1   -1   0
+$EndComp
 $EndSCHEMATC

Commit message: more dabbling
Connections:
- net MTSA: now also R4.2; no longer R4.1
- net ref: now also R4.1; no longer R4.2
Other:
- moved on the sheet: D1, R1, R2, R4, R5, R6, W3, W4, W6
Changed lines of the file:
@@
 L R R4
 U 1 1 58064DD0
-P 3450 5600
-F 0 "R4" V 3530 5600 50  0000 C CNN
-F 1 "10k" V 3450 5600 50  0000 C CNN
-F 2 "Resistors_SMD:R_0603" V 3380 5600 50  0000 L CNN
-F 3 "" H 3450 5600 50  0000 C CNN
-	1    3450 5600
-	0    1    1    0
+P 3600 5750
+F 0 "R4" V 3680 5750 50  0000 C CNN
+F 1 "10k" V 3600 5750 50  0000 C CNN
+F 2 "Resistors_SMD:R_0603" H 3530 5750 50  0000 L CNN
+F 3 "" H 3600 5750 50  0000 C CNN
+	1    3600 5750
+	-1   0    0    1
 $EndComp
 $Comp
 L R R5
 U 1 1 58064FBC
-P 4900 4950
-F 0 "R5" V 4980 4950 50  0000 C CNN
-F 1 "10k" V 4900 4950 50  0000 C CNN
-F 2 "Resistors_SMD:R_0603" V 4830 4950 50  0000 R CNN
-F 3 "" H 4900 4950 50  0000 C CNN
-	1    4900 4950
-	-1   0    0    1
+P 5250 5200
+F 0 "R5" V 5330 5200 50  0000 C CNN
+F 1 "10k" V 5250 5200 50  0000 C CNN
+F 2 "Resistors_SMD:R_0603" V 5180 5200 50  0000 R CNN
+F 3 "" H 5250 5200 50  0000 C CNN
+	1    5250 5200
+	0    -1   -1   0
 $EndComp
 $Comp
 L R R1
 U 1 1 580650CE
-P 2300 5350
-F 0 "R1" V 2380 5350 50  0000 C CNN
-F 1 "100k" V 2300 5350 50  0000 C CNN
-F 2 "Resistors_SMD:R_0603_HandSoldering" H 2230 5350 50  0000 R CNN
-F 3 "" H 2300 5350 50  0000 C CNN
-	1    2300 5350
-	1    0    0    -1
+P 3900 6000
+F 0 "R1" V 3980 6000 50  0000 C CNN
+F 1 "100k" V 3900 6000 50  0000 C CNN
+F 2 "Resistors_SMD:R_0603_HandSoldering" V 4000 5900 50  0000 L TNN
+F 3 "" H 3900 6000 50  0000 C CNN
+	1    3900 6000
+	0    1    1    0
 $EndComp
 $Comp
 L R R2
 U 1 1 580650FF
-P 2300 5850
-F 0 "R2" V 2380 5850 50  0000 C CNN
-F 1 "100k" V 2300 5850 50  0000 C CNN
-F 2 "Resistors_SMD:R_0603_HandSoldering" H 2230 5850 50  0000 R CNN
-F 3 "" H 2300 5850 50  0000 C CNN
-	1    2300 5850
-	1    0    0    -1
+P 3250 6000
+F 0 "R2" V 3330 6000 50  0000 C CNN
+F 1 "100k" V 3250 6000 50  0000 C CNN
+F 2 "Resistors_SMD:R_0603_HandSoldering" V 3180 6000 50  0000 C CNN
+F 3 "" H 3250 6000 50  0000 C CNN
+	1    3250 6000
+	0    1    1    0
 $EndComp
 $Comp
@@
 L R R6
 U 1 1 58065673
-P 5400 5350
-F 0 "R6" V 5480 5350 50  0000 C CNN
-F 1 "1k" V 5400 5350 50  0000 C CNN
-F 2 "Resistors_SMD:R_0603" V 5330 5350 50  0000 R CNN
-F 3 "" H 5400 5350 50  0000 C CNN
-	1    5400 5350
-	1    0    0    -1
+P 5550 5600
+F 0 "R6" V 5630 5600 50  0000 C CNN
+F 1 "1k" V 5550 5600 50  0000 C CNN
+F 2 "Resistors_SMD:R_0603" V 5480 5600 50  0000 R CNN
+F 3 "" H 5550 5600 50  0000 C CNN
+	1    5550 5600
+	0    1    1    0
 $EndComp
 $Comp
 L LED D1
 U 1 1 5806579A
-P 5400 4900
-F 0 "D1" H 5400 5000 50  0000 C CNN
-F 1 "LED" H 5400 4800 50  0000 C CNN
-F 2 "LEDs:LED_1206" H 5400 4900 50  0000 C TNN
-F 3 "" H 5400 4900 50  0000 C CNN
-	1    5400 4900
-	0    -1   -1   0
+P 5900 5600
+F 0 "D1" H 5900 5700 50  0000 C CNN
+F 1 "LED" H 5900 5500 50  0000 C CNN
+F 2 "LEDs:LED_1206" H 5900 5600 50  0000 C TNN
+F 3 "" H 5900 5600 50  0000 C CNN
+	1    5900 5600
+	1    0    0    -1
 $EndComp
 Text Label 4950 5600 0    60   ~ 0
@@
 Text Label 3300 4900 0    60   ~ 0
 sns
-Text Label 2750 5600 0    60   ~ 0
+Text Label 3650 6000 0    60   ~ 0
 ref
 $Comp
 L TEST_1P W6
 U 1 1 580662C8
-P 5100 5200
-F 0 "W6" H 5100 5470 50  0000 C CNN
-F 1 "TEST_MTPM" H 5100 5400 50  0000 C CNN
-F 2 "Measurement_Points:Measurement_Point_Round-SMD-Pad_Small" H 5300 5200 50  0001 C CNN
-F 3 "" H 5300 5200 50  0000 C CNN
-	1    5100 5200
-	0    1    1    0
+P 4900 5100
+F 0 "W6" H 4900 5370 50  0000 C CNN
+F 1 "TEST_MTPM" H 4900 5300 50  0000 C CNN
+F 2 "Measurement_Points:Measurement_Point_Round-SMD-Pad_Small" H 5100 5100 50  0001 C CNN
+F 3 "" H 5100 5100 50  0000 C CNN
+	1    4900 5100
+	1    0    0    -1
 $EndComp
 $Comp
 L VDD #vdd03
 U 1 1 58067C71
-P 5400 4500
-F 0 "#vdd03" H 5400 4350 50  0001 C CNN
-F 1 "VDD" H 5400 4650 50  0000 C CNN
-F 2 "" H 5400 4500 50  0000 C CNN
-F 3 "" H 5400 4500 50  0000 C CNN
-	1    5400 4500
-	1    0    0    -1
+P 6100 5600
+F 0 "#vdd03" H 6100 5450 50  0001 C CNN
+F 1 "VDD" H 6100 5750 50  0000 C CNN
+F 2 "" H 6100 5600 50  0000 C CNN
+F 3 "" H 6100 5600 50  0000 C CNN
+	1    6100 5600
+	0    1    1    0
 $EndComp
 $Comp
 L VDD #vdd04
 U 1 1 580681E5
-P 4900 4600
-F 0 "#vdd04" H 4900 4450 50  0001 C CNN
-F 1 "VDD" H 4900 4750 50  0000 C CNN
-F 2 "" H 4900 4600 50  0000 C CNN
-F 3 "" H 4900 4600 50  0000 C CNN
-	1    4900 4600
-	1    0    0    -1
+P 5400 5200
+F 0 "#vdd04" H 5400 5050 50  0001 C CNN
+F 1 "VDD" H 5400 5350 50  0000 C CNN
+F 2 "" H 5400 5200 50  0000 C CNN
+F 3 "" H 5400 5200 50  0000 C CNN
+	1    5400 5200
+	0    1    1    0
 $EndComp
 $Comp
@@
 L VDD #vdd06
 U 1 1 58068249
-P 2300 5100
-F 0 "#vdd06" H 2300 4950 50  0001 C CNN
-F 1 "VDD" H 2300 5250 50  0000 C CNN
-F 2 "" H 2300 5100 50  0000 C CNN
-F 3 "" H 2300 5100 50  0000 C CNN
-	1    2300 5100
-	1    0    0    -1
+P 4050 6000
+F 0 "#vdd06" H 4050 5850 50  0001 C CNN
+F 1 "VDD" H 4050 6150 50  0000 C CNN
+F 2 "" H 4050 6000 50  0000 C CNN
+F 3 "" H 4050 6000 50  0000 C CNN
+	1    4050 6000
+	0    1    1    0
 $EndComp
 $Comp
@@
 L GND #gnd08
 U 1 1 580686F1
-P 2300 6100
-F 0 "#gnd08" H 2300 5850 50  0001 C CNN
-F 1 "GND" H 2300 5950 50  0000 C CNN
-F 2 "" H 2300 6100 50  0000 C CNN
-F 3 "" H 2300 6100 50  0000 C CNN
-	1    2300 6100
-	1    0    0    -1
+P 3100 6000
+F 0 "#gnd08" H 3100 5750 50  0001 C CNN
+F 1 "GND" H 3100 5850 50  0000 C CNN
+F 2 "" H 3100 6000 50  0000 C CNN
+F 3 "" H 3100 6000 50  0000 C CNN
+	1    3100 6000
+	0    1    1    0
 $EndComp
 $Comp
@@
 	4700 5200 5100 5200
 Wire Wire Line
-	2300 5500 2300 5700
-Wire Wire Line
-	2300 5600 3300 5600
-Connection ~ 2300 5600
-Wire Wire Line
-	2300 5100 2300 5200
-Wire Wire Line
-	2300 6000 2300 6100
-Wire Wire Line
-	5400 5600 5400 5500
-Wire Wire Line
-	5400 5100 5400 5200
-Wire Wire Line
-	5400 4500 5400 4700
-Wire Wire Line
-	4700 5600 5500 5600
-Connection ~ 5400 5600
-Wire Wire Line
-	4900 4600 4900 4800
+	4700 5600 5400 5600
 Wire Wire Line
 	4900 5100 4900 5200
 Connection ~ 4900 5200
-Wire Wire Line
-	2900 5600 2900 5600
-Connection ~ 2900 5600
 Wire Wire Line
 	7150 2800 7000 2800
@@
 Wire Wire Line
 	3600 5600 3900 5600
-Wire Wire Line
-	2900 5400 2900 5600
 $Comp
 L SEW_1X2 W3
 U 1 1 580A30E6
-P 2900 5400
-F 0 "W3" H 2900 5670 50  0000 C CNN
-F 1 "sa" H 2900 5600 50  0000 C CNN
-F 2 "buttons:sew_1x2" H 3100 5400 50  0000 C CNN
-F 3 "" H 3100 5400 50  0000 C CNN
-	1    2900 5400
-	1    0    0    -1
+P 3600 6100
+F 0 "W3" H 3600 6370 50  0000 C CNN
+F 1 "sa" H 3600 6300 50  0000 C CNN
+F 2 "buttons:sew_1x2" H 3700 6450 50  0000 C CNN
+F 3 "" H 3800 6100 50  0000 C CNN
+	1    3600 6100
+	-1   0    0    1
 $EndComp
 $Comp
 L SEW_1X2 W4
 U 1 1 580A3684
-P 5500 5600
-F 0 "W4" H 5500 5870 50  0000 C CNN
-F 1 "out" H 5500 5800 50  0000 C CNN
-F 2 "buttons:sew_1x2" H 5700 5600 50  0000 C CNN
-F 3 "" H 5700 5600 50  0000 C CNN
-	1    5500 5600
-	0    1    1    0
+P 4950 5800
+F 0 "W4" H 4950 6070 50  0000 C CNN
+F 1 "out" H 4950 6000 50  0000 C CNN
+F 2 "buttons:sew_1x2" H 5150 5800 50  0000 C CNN
+F 3 "" H 5150 5800 50  0000 C CNN
+	1    4950 5800
+	-1   0    0    1
 $EndComp
 $Comp
@@
 	0    -1   -1   0
 $EndComp
+Wire Wire Line
+	4950 5800 4950 5600
+Connection ~ 4950 5600
+Wire Wire Line
+	3600 5900 3600 6100
+Wire Wire Line
+	3400 6000 3750 6000
+Connection ~ 3600 6000
+$Comp
+L GND #gnd011
+U 1 1 580A55A8
+P 4200 4850
+F 0 "#gnd011" H 4200 4600 50  0001 C CNN
+F 1 "GND" H 4200 4700 50  0000 C CNN
+F 2 "" H 4200 4850 50  0000 C CNN
+F 3 "" H 4200 4850 50  0000 C CNN
+	1    4200 4850
+	-1   0    0    1
+$EndComp
+Wire Wire Line
+	3900 5400 4200 5400
+Wire Wire Line
+	4200 5400 4200 4850
+$Comp
+L VDD #vdd012
+U 1 1 580A5607
+P 4400 5800
+F 0 "#vdd012" H 4400 5650 50  0001 C CNN
+F 1 "VDD" H 4400 5950 50  0000 C CNN
+F 2 "" H 4400 5800 50  0000 C CNN
+F 3 "" H 4400 5800 50  0000 C CNN
+	1    4400 5800
+	-1   0    0    1
+$EndComp
+Wire Wire Line
+	4700 5400 4400 5400
+Wire Wire Line
+	4400 5400 4400 5800
 $EndSCHEMATC
