File: wearables/kicad/MTCH101_Disc.sch (KiCad schematic (older format))
At the start: 15 parts, among them U1 MTCH101_PKG

Commit message: More misc play.
Parts:
- added P1: TST1, Connect:PINHEAD1-2, symbol CONN_01X02
- added P2: TST2, Connect:PINHEAD1-2, symbol CONN_01X02
- added P3: TST3, Connect:PINHEAD1-2, symbol CONN_01X02
- added P4: TST4, Connect:PINHEAD1-2, symbol CONN_01X02
- added W10: TST2B, buttons:sew_2x2, symbol SEW_2X2
- added W11: TST3A, buttons:lego_1x2, symbol SEW_1X2
- added W12: TST3B, buttons:lego_1x2, symbol SEW_1X2
- added W13: TST4A, buttons:lego_2x2, symbol SEW_2X2
- added W14: TST4B, buttons:lego_2x2, symbol SEW_2X2
- added W7: TST1A, buttons:sew_1x2, symbol SEW_1X2
- added W8: TST1B, buttons:sew_1x2, symbol SEW_1X2
- added W9: TST2A, buttons:sew_2x2, symbol SEW_2X2
Connections:
- new net tst1a: P1.1 (P1), W7.1
- new net tst1b: P1.2 (P2), W8.1
- new net tst2a: P2.1 (P1), W9.1
- new net tst2b: P2.2 (P2), W10.1
- new net tst3a: P3.1 (P1), W11.1
- new net tst3b: P3.2 (P2), W12.1
- new net tst4a: P4.1 (P1), W13.1
- new net tst4b: P4.2 (P2), W14.1
Changed lines of the file:
@@
 Wire Wire Line
 	4400 5400 4400 5800
+Wire Notes Line
+	4100 1200 1350 1200
+Wire Notes Line
+	1350 1200 1350 2700
+Wire Notes Line
+	1350 2700 4100 2700
+Wire Notes Line
+	4100 2700 4100 1200
+$Comp
+L SEW_1X2 W7
+U 1 1 580CE257
+P 1600 1600
+F 0 "W7" H 1600 1870 50  0000 C CNN
+F 1 "TST1A" H 1600 1800 50  0000 C CNN
+F 2 "buttons:sew_1x2" H 1800 1600 50  0000 C CNN
+F 3 "" H 1800 1600 50  0000 C CNN
+	1    1600 1600
+	1    0    0    -1
+$EndComp
+$Comp
+L SEW_1X2 W8
+U 1 1 580CE2C7
+P 1600 2300
+F 0 "W8" H 1600 2570 50  0000 C CNN
+F 1 "TST1B" H 1600 2500 50  0000 C CNN
+F 2 "buttons:sew_1x2" H 1800 2300 50  0000 C CNN
+F 3 "" H 1800 2300 50  0000 C CNN
+	1    1600 2300
+	-1   0    0    1
+$EndComp
+$Comp
+L SEW_2X2 W9
+U 1 1 580CE33E
+P 2000 1600
+F 0 "W9" H 2000 1870 50  0000 C CNN
+F 1 "TST2A" H 2000 1800 50  0000 C CNN
+F 2 "buttons:sew_2x2" H 2200 1600 50  0000 C CNN
+F 3 "" H 2200 1600 50  0000 C CNN
+	1    2000 1600
+	1    0    0    -1
+$EndComp
+$Comp
+L SEW_2X2 W10
+U 1 1 580CE39E
+P 2000 2300
+F 0 "W10" H 2000 2570 50  0000 C CNN
+F 1 "TST2B" H 2000 2500 50  0000 C CNN
+F 2 "buttons:sew_2x2" H 2200 2300 50  0000 C CNN
+F 3 "" H 2200 2300 50  0000 C CNN
+	1    2000 2300
+	-1   0    0    1
+$EndComp
+Wire Wire Line
+	1600 1600 1600 1900
+Wire Wire Line
+	2000 1600 2000 1900
+Wire Wire Line
+	2000 2000 2000 2300
+Wire Wire Line
+	1600 2000 1600 2300
+$Comp
+L CONN_01X02 P1
+U 1 1 580CE890
+P 1800 1950
+F 0 "P1" H 1800 2100 50  0000 C CNN
+F 1 "TST1" V 1900 1950 50  0000 C CNN
+F 2 "Connect:PINHEAD1-2" H 1800 1950 50  0000 C CNN
+F 3 "" H 1800 1950 50  0000 C CNN
+	1    1800 1950
+	1    0    0    -1
+$EndComp
+$Comp
+L CONN_01X02 P2
+U 1 1 580CE8EA
+P 2200 1950
+F 0 "P2" H 2200 2100 50  0000 C CNN
+F 1 "TST2" V 2300 1950 50  0000 C CNN
+F 2 "Connect:PINHEAD1-2" H 2200 1950 50  0000 C CNN
+F 3 "" H 2200 1950 50  0000 C CNN
+	1    2200 1950
+	1    0    0    -1
+$EndComp
+$Comp
+L SEW_1X2 W11
+U 1 1 580CF0AD
+P 3000 1600
+F 0 "W11" H 3000 1870 50  0000 C CNN
+F 1 "TST3A" H 3000 1800 50  0000 C CNN
+F 2 "buttons:lego_1x2" H 3200 1600 50  0000 C CNN
+F 3 "" H 3200 1600 50  0000 C CNN
+	1    3000 1600
+	1    0    0    -1
+$EndComp
+$Comp
+L SEW_1X2 W12
+U 1 1 580CF0B3
+P 3000 2300
+F 0 "W12" H 3000 2570 50  0000 C CNN
+F 1 "TST3B" H 3000 2500 50  0000 C CNN
+F 2 "buttons:lego_1x2" H 3200 2300 50  0000 C CNN
+F 3 "" H 3200 2300 50  0000 C CNN
+	1    3000 2300
+	-1   0    0    1
+$EndComp
+$Comp
+L SEW_2X2 W13
+U 1 1 580CF0B9
+P 3400 1600
+F 0 "W13" H 3400 1870 50  0000 C CNN
+F 1 "TST4A" H 3400 1800 50  0000 C CNN
+F 2 "buttons:lego_2x2" H 3600 1600 50  0000 C CNN
+F 3 "" H 3600 1600 50  0000 C CNN
+	1    3400 1600
+	1    0    0    -1
+$EndComp
+$Comp
+L SEW_2X2 W14
+U 1 1 580CF0BF
+P 3400 2300
+F 0 "W14" H 3400 2570 50  0000 C CNN
+F 1 "TST4B" H 3400 2500 50  0000 C CNN
+F 2 "buttons:lego_2x2" H 3600 2300 50  0000 C CNN
+F 3 "" H 3600 2300 50  0000 C CNN
+	1    3400 2300
+	-1   0    0    1
+$EndComp
+Wire Wire Line
+	3000 1600 3000 1900
+Wire Wire Line
+	3400 1600 3400 1900
+Wire Wire Line
+	3400 2000 3400 2300
+Wire Wire Line
+	3000 2000 3000 2300
+$Comp
+L CONN_01X02 P3
+U 1 1 580CF0C9
+P 3200 1950
+F 0 "P3" H 3200 2100 50  0000 C CNN
+F 1 "TST3" V 3300 1950 50  0000 C CNN
+F 2 "Connect:PINHEAD1-2" H 3200 1950 50  0000 C CNN
+F 3 "" H 3200 1950 50  0000 C CNN
+	1    3200 1950
+	1    0    0    -1
+$EndComp
+$Comp
+L CONN_01X02 P4
+U 1 1 580CF0CF
+P 3600 1950
+F 0 "P4" H 3600 2100 50  0000 C CNN
+F 1 "TST4" V 3700 1950 50  0000 C CNN
+F 2 "Connect:PINHEAD1-2" H 3600 1950 50  0000 C CNN
+F 3 "" H 3600 1950 50  0000 C CNN
+	1    3600 1950
+	1    0    0    -1
+$EndComp
+Text Label 1600 1700 0    60   ~ 0
+tst1a
+Text Label 1600 2150 0    60   ~ 0
+tst1b
+Text Label 2000 1700 0    60   ~ 0
+tst2a
+Text Label 2000 2150 0    60   ~ 0
+tst2b
+Text Label 3000 1700 0    60   ~ 0
+tst3a
+Text Label 3000 2200 0    60   ~ 0
+tst3b
+Text Label 3400 1750 0    60   ~ 0
+tst4a
+Text Label 3400 2200 0    60   ~ 0
+tst4b
 $EndSCHEMATC
